Commit message: Update arctos.urdf.xacro

File: ROS2/src/arctos_urdf_description/urdf/arctos.urdf.xacro (robot description, xacro)
@@ -1,497 +1,261 @@
-<?xml version="1.0" encoding="utf-8" ?>
-<!-- =================================================================================== -->
-<!-- |    This document was autogenerated by xacro from /home/aa/arctos_ros/src/arctos_urdf_description/urdf/arctos_urdf.xacro | -->
-<!-- |    EDITING THIS FILE BY HAND IS NOT RECOMMENDED                                 | -->
-<!-- =================================================================================== -->
-<robot name="arctos_urdf">
-    <material name="silver_default">
-        <color rgba="0.700 0.700 0.700 1.000" />
-    </material>
-    <material name="paint_metallic_blue_2">
-        <color rgba="0.7764705882352941 0.7764705882352941 0.7764705882352941 1.0" />
-    </material>
-    <transmission name="Revolute 21_tran">
-        <type>transmission_interface/SimpleTransmission</type>
-        <joint name="Revolute 21">
-            <hardwareInterface>hardware_interface/EffortJointInterface</hardwareInterface>
-        </joint>
-        <actuator name="Revolute 21_actr">
-            <hardwareInterface>hardware_interface/EffortJointInterface</hardwareInterface>
-            <mechanicalReduction>1</mechanicalReduction>
-        </actuator>
-    </transmission>
-    <transmission name="Revolute 22_tran">
-        <type>transmission_interface/SimpleTransmission</type>
-        <joint name="Revolute 22">
-            <hardwareInterface>hardware_interface/EffortJointInterface</hardwareInterface>
-        </joint>
-        <actuator name="Revolute 22_actr">
-            <hardwareInterface>hardware_interface/EffortJointInterface</hardwareInterface>
-            <mechanicalReduction>1</mechanicalReduction>
-        </actuator>
-    </transmission>
-    <transmission name="Revolute 23_tran">
-        <type>transmission_interface/SimpleTransmission</type>
-        <joint name="Revolute 23">
-            <hardwareInterface>hardware_interface/EffortJointInterface</hardwareInterface>
-        </joint>
-        <actuator name="Revolute 23_actr">
-            <hardwareInterface>hardware_interface/EffortJointInterface</hardwareInterface>
-            <mechanicalReduction>1</mechanicalReduction>
-        </actuator>
-    </transmission>
-    <transmission name="Revolute 24_tran">
-        <type>transmission_interface/SimpleTransmission</type>
-        <joint name="Revolute 24">
-            <hardwareInterface>hardware_interface/EffortJointInterface</hardwareInterface>
-        </joint>
-        <actuator name="Revolute 24_actr">
-            <hardwareInterface>hardware_interface/EffortJointInterface</hardwareInterface>
-            <mechanicalReduction>1</mechanicalReduction>
-        </actuator>
-    </transmission>
-    <transmission name="Revolute 25_tran">
-        <type>transmission_interface/SimpleTransmission</type>
-        <joint name="Revolute 25">
-            <hardwareInterface>hardware_interface/EffortJointInterface</hardwareInterface>
-        </joint>
-        <actuator name="Revolute 25_actr">
-            <hardwareInterface>hardware_interface/EffortJointInterface</hardwareInterface>
-            <mechanicalReduction>1</mechanicalReduction>
-        </actuator>
-    </transmission>
-    <transmission name="Revolute 27_tran">
-        <type>transmission_interface/SimpleTransmission</type>
-        <joint name="Revolute 27">
-            <hardwareInterface>hardware_interface/EffortJointInterface</hardwareInterface>
-        </joint>
-        <actuator name="Revolute 27_actr">
-            <hardwareInterface>hardware_interface/EffortJointInterface</hardwareInterface>
-            <mechanicalReduction>1</mechanicalReduction>
-        </actuator>
-    </transmission>
-    <transmission name="Slider 28_tran">
-        <type>transmission_interface/SimpleTransmission</type>
-        <joint name="Slider 28">
-            <hardwareInterface>hardware_interface/EffortJointInterface</hardwareInterface>
-        </joint>
-        <actuator name="Slider 28_actr">
-            <hardwareInterface>hardware_interface/EffortJointInterface</hardwareInterface>
-            <mechanicalReduction>1</mechanicalReduction>
-        </actuator>
-    </transmission>
-    <transmission name="Slider 29_tran">
-        <type>transmission_interface/SimpleTransmission</type>
-        <joint name="Slider 29">
-            <hardwareInterface>hardware_interface/EffortJointInterface</hardwareInterface>
-        </joint>
-        <actuator name="Slider 29_actr">
-            <hardwareInterface>hardware_interface/EffortJointInterface</hardwareInterface>
-            <mechanicalReduction>1</mechanicalReduction>
-        </actuator>
-    </transmission>
-    <gazebo>
-        <plugin filename="libgazebo_ros_control.so" name="control" />
-    </gazebo>
-    <gazebo reference="base_link">
-        <material>Gazebo/Silver</material>
-        <mu1>0.2</mu1>
-        <mu2>0.2</mu2>
-        <selfCollide>true</selfCollide>
-        <gravity>true</gravity>
-    </gazebo>
-    <gazebo reference="Link_1_1">
-        <material>Gazebo/Silver</material>
-        <mu1>0.2</mu1>
-        <mu2>0.2</mu2>
-        <selfCollide>true</selfCollide>
-    </gazebo>
-    <gazebo reference="Link_2_1">
-        <material>Gazebo/Silver</material>
-        <mu1>0.2</mu1>
-        <mu2>0.2</mu2>
-        <selfCollide>true</selfCollide>
-    </gazebo>
-    <gazebo reference="Link_3_1">
-        <material>Gazebo/Silver</material>
-        <mu1>0.2</mu1>
-        <mu2>0.2</mu2>
-        <selfCollide>true</selfCollide>
-    </gazebo>
-    <gazebo reference="Link_4_1">
-        <material>Gazebo/Silver</material>
-        <mu1>0.2</mu1>
-        <mu2>0.2</mu2>
-        <selfCollide>true</selfCollide>
-    </gazebo>
-    <gazebo reference="Link_5_1">
-        <material>Gazebo/Silver</material>
-        <mu1>0.2</mu1>
-        <mu2>0.2</mu2>
-        <selfCollide>true</selfCollide>
-    </gazebo>
-    <gazebo reference="Gripper_1">
-        <material>Gazebo/Silver</material>
-        <mu1>0.2</mu1>
-        <mu2>0.2</mu2>
-        <selfCollide>true</selfCollide>
-    </gazebo>
-    <gazebo reference="Link_6_1">
-        <material>Gazebo/Silver</material>
-        <mu1>0.2</mu1>
-        <mu2>0.2</mu2>
-        <selfCollide>true</selfCollide>
-    </gazebo>
-    <gazebo reference="Left_jaw_1">
-        <material>Gazebo/Silver</material>
-        <mu1>0.2</mu1>
-        <mu2>0.2</mu2>
-        <selfCollide>true</selfCollide>
-    </gazebo>
-    <gazebo reference="Right_jaw_1">
-        <material>Gazebo/Silver</material>
-        <mu1>0.2</mu1>
-        <mu2>0.2</mu2>
-        <selfCollide>true</selfCollide>
-    </gazebo>
-    <link name="base_link">
-<inertial>
-            <origin rpy="0 0 0" xyz="0.0009375030874740357 0.047087016508753216 0.06663230338123677" />
-            <mass value="7.598577592821282" />
-            <inertia ixx="0.063328" ixy="-0.000434" ixz="0.000108" iyy="0.03095" iyz="0.001366" izz="0.072371" />
-        </inertial>
-        <visual>
-            <origin rpy="0 0 0" xyz="0 0 0" />
-            <geometry>
-                <mesh filename="package://arctos_urdf_description/meshes/base_link.stl" scale="0.001 0.001 0.001" />
-            </geometry>
-            <material name="paint_metallic_blue_2" />
-        </visual>
-        <collision>
-            <origin rpy="0 0 0" xyz="0 0 0" />
-            <geometry>
-                <mesh filename="package://arctos_urdf_description/meshes/base_link.stl" scale="0.001 0.001 0.001" />
-            </geometry>
-        </collision>
-    </link>
-    <link name="Link_1_1">
-<inertial>
-            <origin rpy="0 0 0" xyz="0.0022188890353287776 -0.004863444449475237 0.08546835509394825" />
-            <mass value="10.394711633971145" />
-            <inertia ixx="0.061139" ixy="0.00017" ixz="-0.00148" iyy="0.073854" iyz="0.003835" izz="0.05669" />
-        </inertial>
-        <visual>
-            <origin rpy="0 0 0" xyz="-0.0 -0.000529 -0.111" />
-            <geometry>
-                <mesh filename="package://arctos_urdf_description/meshes/Link_1_1.stl" scale="0.001 0.001 0.001" />
-            </geometry>
-            <material name="paint_metallic_blue_2" />
-        </visual>
-        <collision>
-            <origin rpy="0 0 0" xyz="-0.0 -0.000529 -0.111" />
-            <geometry>
-                <mesh filename="package://arctos_urdf_description/meshes/Link_1_1.stl" scale="0.001 0.001 0.001" />
-            </geometry>
-        </collision>
-    </link>
-    <link name="Link_2_1">
-<inertial>
-            <origin rpy="0 0 0" xyz="0.055314283466519745 0.010843565259072822 0.11412354328486207" />
-            <mass value="11.558090086674309" />
-            <inertia ixx="0.128567" ixy="3e-06" ixz="0.001539" iyy="0.14463" iyz="-0.003293" izz="0.044463" />
-        </inertial>
-        <visual>
-            <origin rpy="0 0 0" xyz="0.05713 0.020356 -0.289378" />
-            <geometry>
-                <mesh filename="package://arctos_urdf_description/meshes/Link_2_1.stl" scale="0.001 0.001 0.001" />
-            </geometry>
-            <material name="paint_metallic_blue_2" />
-        </visual>
-        <collision>
-            <origin rpy="0 0 0" xyz="0.05713 0.020356 -0.289378" />
-            <geometry>
-                <mesh filename="package://arctos_urdf_description/meshes/Link_2_1.stl" scale="0.001 0.001 0.001" />
-            </geometry>
-        </collision>
-    </link>
-    <link name="Link_3_1">
-<inertial>
-            <origin rpy="0 0 0" xyz="-0.04178369242643258 -0.03913025368943244 0.01221763827191602" />
-            <mass value="3.601405589552794" />
-            <inertia ixx="0.012497" ixy="-3.6e-05" ixz="-8.1e-05" iyy="0.006916" iyz="0.001536" izz="0.011789" />
-        </inertial>
-        <visual>
-            <origin rpy="0 0 0" xyz="-0.043 0.019045 -0.550385" />
-            <geometry>
-                <mesh filename="package://arctos_urdf_description/meshes/Link_3_1.stl" scale="0.001 0.001 0.001" />
-            </geometry>
-            <material name="paint_metallic_blue_2" />
-        </visual>
-        <collision>
-            <origin rpy="0 0 0" xyz="-0.043 0.019045 -0.550385" />
-            <geometry>
-                <mesh filename="package://arctos_urdf_description/meshes/Link_3_1.stl" scale="0.001 0.001 0.001" />
-            </geometry>
-        </collision>
-    </link>
-    <link name="Link_4_1">
-<inertial>
-            <origin rpy="0 0 0" xyz="0.00021104999825562586 -0.06028834880207104 -0.0005408226217131773" />
-            <mass value="3.7852887653107565" />
-            <inertia ixx="0.011624" ixy="-9e-06" ixz="4e-06" iyy="0.011491" iyz="-7.1e-05" izz="0.017363" />
-        </inertial>
-        <visual>
-            <origin rpy="0 0 0" xyz="-1e-06 0.15874 -0.57209" />
-            <geometry>
-                <mesh filename="package://arctos_urdf_description/meshes/Link_4_1.stl" scale="0.001 0.001 0.001" />
-            </geometry>
-            <material name="paint_metallic_blue_2" />
-        </visual>
-        <collision>
-            <origin rpy="0 0 0" xyz="-1e-06 0.15874 -0.57209" />
-            <geometry>
-                <mesh filename="package://arctos_urdf_description/meshes/Link_4_1.stl" scale="0.001 0.001 0.001" />
-            </geometry>
-        </collision>
-    </link>
-    <link name="Link_5_1">
-<inertial>
-            <origin rpy="0 0 0" xyz="0.0397291414278933 -0.012662394123331089 0.0007929187272999183" />
-            <mass value="0.8319811655030993" />
-            <inertia ixx="0.000732" ixy="-1.2e-05" ixz="5e-06" iyy="0.000958" iyz="-5e-06" izz="0.000907" />
-        </inertial>
-        <visual>
-            <origin rpy="0 0 0" xyz="0.039011 0.279927 -0.570316" />
-            <geometry>
-                <mesh filename="package://arctos_urdf_description/meshes/Link_5_1.stl" scale="0.001 0.001 0.001" />
-            </geometry>
-            <material name="paint_metallic_blue_2" />
-        </visual>
-        <collision>
-            <origin rpy="0 0 0" xyz="0.039011 0.279927 -0.570316" />
-            <geometry>
-                <mesh filename="package://arctos_urdf_description/meshes/Link_5_1.stl" scale="0.001 0.001 0.001" />
-            </geometry>
-        </collision>
-    </link>
-    <link name="Gripper_1">
-<inertial>
-            <origin rpy="0 0 0" xyz="0.0036112727264542635 -0.014760653808445767 -0.00103677815369696" />
-            <mass value="0.5810486809925093" />
-            <inertia ixx="0.000385" ixy="1e-05" ixz="3e-06" iyy="0.000495" iyz="-2e-06" izz="0.000263" />
-        </inertial>
-        <visual>
-            <origin rpy="0 0 0" xyz="-0.000193 0.319847 -0.570316" />
-            <geometry>
-                <mesh filename="package://arctos_urdf_description/meshes/Gripper_1.stl" scale="0.001 0.001 0.001" />
-            </geometry>
-            <material name="paint_metallic_blue_2" />
-        </visual>
-        <collision>
-            <origin rpy="0 0 0" xyz="-0.000193 0.319847 -0.570316" />
-            <geometry>
-                <mesh filename="package://arctos_urdf_description/meshes/Gripper_1.stl" scale="0.001 0.001 0.001" />
-            </geometry>
-        </collision>
-    </link>
-    <link name="Link_6_1">
-<inertial>
-            <origin rpy="0 0 0" xyz="6.567946382108388e-08 -0.003042398377876454 -3.032508957279134e-07" />
-            <mass value="0.10343478090890781" />
-            <inertia ixx="5.2e-05" ixy="-0.0" ixz="0.0" iyy="0.000103" iyz="0.0" izz="5.2e-05" />
-        </inertial>
-        <visual>
-            <origin rpy="0 0 0" xyz="-0.000193 0.313762 -0.570316" />
-            <geometry>
-                <mesh filename="package://arctos_urdf_description/meshes/Link_6_1.stl" scale="0.001 0.001 0.001" />
-            </geometry>
-            <material name="paint_metallic_blue_2" />
-        </visual>
-        <collision>
-            <origin rpy="0 0 0" xyz="-0.000193 0.313762 -0.570316" />
-            <geometry>
-                <mesh filename="package://arctos_urdf_description/meshes/Link_6_1.stl" scale="0.001 0.001 0.001" />
-            </geometry>
-        </collision>
-    </link>
-    <link name="Left_jaw_1">
-<inertial>
-            <origin rpy="0 0 0" xyz="-0.011142702480351952 -0.009692440309284511 -0.009385792627785827" />
-            <mass value="0.07369602565859415" />
-            <inertia ixx="1.1e-05" ixy="2e-06" ixz="-0.0" iyy="6e-06" iyz="-0.0" izz="1.4e-05" />
-        </inertial>
-        <visual>
-            <origin rpy="0 0 0" xyz="-0.007934 0.359845 -0.599867" />
-            <geometry>
-                <mesh filename="package://arctos_urdf_description/meshes/Left_jaw_1.stl" scale="0.001 0.001 0.001" />
-            </geometry>
-            <material name="paint_metallic_blue_2" />
-        </visual>
-        <collision>
-            <origin rpy="0 0 0" xyz="-0.007934 0.359845 -0.599867" />
-            <geometry>
-                <mesh filename="package://arctos_urdf_description/meshes/Left_jaw_1.stl" scale="0.001 0.001 0.001" />
-            </geometry>
-        </collision>
-    </link>
-    <link name="Right_jaw_1">
-<inertial>
-            <origin rpy="0 0 0" xyz="-0.008289104952972526 -0.009768535307719373 0.009395511902715814" />
-            <mass value="0.07312902168719511" />
-            <inertia ixx="1.1e-05" ixy="-1e-06" ixz="-1e-06" iyy="6e-06" iyz="0.0" izz="1.4e-05" />
-        </inertial>
-        <visual>
-            <origin rpy="0 0 0" xyz="-0.007934 0.359845 -0.539867" />
-            <geometry>
-                <mesh filename="package://arctos_urdf_description/meshes/Right_jaw_1.stl" scale="0.001 0.001 0.001" />
-            </geometry>
-            <material name="paint_metallic_blue_2" />
-        </visual>
-        <collision>
-            <origin rpy="0 0 0" xyz="-0.007934 0.359845 -0.539867" />
-            <geometry>
-                <mesh filename="package://arctos_urdf_description/meshes/Right_jaw_1.stl" scale="0.001 0.001 0.001" />
-            </geometry>
-        </collision>
-    </link>
-    <joint name="joint1" type="continuous">
-        <origin rpy="0 0 0" xyz="0.0 0.000529 0.111" />
-        <parent link="base_link" />
-        <child link="Link_1_1" />
-        <axis xyz="-0.0 0.0 1.0" />
-    </joint>
-    <joint name="joint2" type="continuous">
-        <origin rpy="0 0 0" xyz="-0.05713 -0.020885 0.178378" />
-        <parent link="Link_1_1" />
-        <child link="Link_2_1" />
-        <axis xyz="1.0 -0.0 -0.0" />
-    </joint>
-    <joint name="joint3" type="continuous">
-        <origin rpy="0 0 0" xyz="0.10013 0.001311 0.261007" />
-        <parent link="Link_2_1" />
-        <child link="Link_3_1" />
-        <axis xyz="-1.0 -0.0 0.0" />
-    </joint>
-    <joint name="joint4" type="continuous">
-        <origin rpy="0 0 0" xyz="-0.042999 -0.139695 0.021705" />
-        <parent link="Link_3_1" />
-        <child link="Link_4_1" />
-        <axis xyz="-0.0 1.0 -0.0" />
-    </joint>
-    <joint name="joint5" type="continuous">
-        <origin rpy="0 0 0" xyz="-0.039012 -0.121187 -0.001774" />
-        <parent link="Link_4_1" />
-        <child link="Link_5_1" />
-        <axis xyz="-1.0 -0.0 0.0" />
-    </joint>
-    <joint name="gripper" type="fixed">
-        <origin rpy="0 0 0" xyz="0.0 -0.006085 0.0" />
-        <parent link="Link_6_1" />
-        <child link="Gripper_1" />
-    </joint>
-    <joint name="joint6" type="continuous">
-        <origin rpy="0 0 0" xyz="0.039204 -0.033835 0.0" />
-        <parent link="Link_5_1" />
-        <child link="Link_6_1" />
-        <axis xyz="-0.0 1.0 -0.0" />
-    </joint>
-    <joint name="jaw1" type="prismatic">
-        <origin rpy="0 0 0" xyz="0.007741 -0.039998 0.029551" />
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